File: AcousticsSingleChannel.kicad_pcb (KiCad board)
At the start: 4 copper layers, 25.6 x 52.2 mm, 59 parts, among them J5 87233-3, J7 SAMTEC-SMH-103-02-X-S, J8 22-05-3021, SW1 416131160803, SW2 Switch_Omron_A6S-1104-PH_eec, U1 OPA1604AIPWR, U2 OPA1604AIPWR, U3 LTC6910-3CTS8#TRPBF, U4 LTC1197LIMS8#PBF

Commit message: Fix various net and footprint issues
Parts:
- ? (x6): footprint AltiumImports: -> AltiumImports:Probepoint
Connections:
- net /BBA IN renamed /BufferBiasAmp/BBA_IN
- ? pad 7: Amp_Out -> /OutputAmplifier/Amp_Out
- C8 pad 2: /BPF OUT -> /Band Pass Filter/BPF_OUT
- R1 pad 2: /BBA OUT -> /BufferBiasAmp/BBA_OUT
- R13 pad 2: /BPF OUT -> /Band Pass Filter/BPF_OUT
- R8 pad 1: /BBA OUT -> /BufferBiasAmp/BBA_OUT
- U1 pad 8: /BBA OUT -> /BufferBiasAmp/BBA_OUT
- U2 pad 5: /Amp_Out -> /OutputAmplifier/Amp_Out
- U2 pad 8: /BPF OUT -> /Band Pass Filter/BPF_OUT
- U3 pad 1: /Amp_Out -> /OutputAmplifier/Amp_Out
- U3 pad 3: /BPF OUT -> /Band Pass Filter/BPF_OUT
Routing:
- net F1_Out: track 28.7 -> 0.00 mm
- net /Band Pass Filter/F1_Out: track 0.00 -> 28.2 mm
- net F3_Out: track 23.0 -> 0.00 mm
- net /Band Pass Filter/F3_Out: track 0.00 -> 22.7 mm
- net BPF OUT: track 15.9 -> 0.00 mm, vias 1 -> 0
- net /OutputAmplifier/Amp_Out: track 0.00 -> 15.9 mm
- net Amp_Out: track 15.4 -> 0.00 mm
- net /Band Pass Filter/BPF_OUT: track 0.00 -> 15.3 mm, vias 0 -> 1
- net BBA OUT: track 8.69 -> 0.00 mm
- net F2_Out: track 8.14 -> 0.00 mm
- net /Band Pass Filter/F2_Out: track 0.00 -> 8.01 mm
- net /BufferBiasAmp/BBA_OUT: track 0.00 -> 7.68 mm
- net VCC: track 42.0 -> 40.7 mm
- net AGND: track 27.7 -> 26.7 mm
- net Net-(J7-CLK): track 13.6 -> 12.9 mm
Other:
- rule pad_to_mask_clearance: 0 -> 0.05

Commit message: Fix logos
Parts:
- added G***: LOGO, LOGO, B.Cu at (148.4, 86.0)
- added G***: LOGO, LOGO, B.Cu at (156.0, 127.3)
- added G***: LOGO, LOGO, B.Cu at (147.7, 127.3)

Commit message: Update fixing local weirdness? Changed some trace widths
Parts:
- removed J7: SAMTEC-SMH-103-02-X-S, AltiumImports:SAMTEC-SMH-103-02-X-S
- removed R18, R19, R20: 10k, AltiumImports:SMD-0603-RES
- removed SW1: 416131160803, AltiumImports:416131160803
- added J1: 87233-3, AltiumImports:TE_87233-3, F.Cu at (156.5, 110.5)
- added J2: 87233-3, AltiumImports:TE_87233-3, F.Cu at (156.5, 120.7)
- moved G*** 9.58 mm to (150.0, 119.8)
- moved C15 9.30 mm to (155.0, 105.2), turned to 0 degrees
- moved G*** 8.35 mm to (144.1, 119.8)
- moved J3 7.78 mm to (156.5, 100.4)
- moved R17 7.35 mm to (150.7, 113.2), turned to 90 degrees
- moved C14 5.45 mm to (153.9, 96.4), turned to 90 degrees
- moved R15 3.64 mm to (153.7, 107.0)
- moved ? 1.57 mm to (147.1, 93.9)
- moved R27 1.52 mm to (140.7, 119.8), turned to 90 degrees
- moved ? 1.31 mm to (147.4, 98.0)
- moved R12 0.74 mm to (153.1, 100.9)
- moved R26 0.63 mm to (137.6, 119.8), turned to -90 degrees
- moved C10 0.61 mm to (153.7, 109.6)
- moved C3 0.12 mm to (156.2, 92.3)
- moved U3 0.10 mm to (148.4, 116.9)
- renumbered J5 to J3
Connections:
- U3 pad 5: /OutputAmplifier/G0 -> /OutputAmplifier/G0_out
- U3 pad 6: /OutputAmplifier/G1 -> /OutputAmplifier/G1_out
- U3 pad 7: /OutputAmplifier/G2 -> /OutputAmplifier/G2_out
Routing:
- net /OutputAmplifier/G2_out: track 0.00 -> 17.4 mm
- net /OutputAmplifier/G1_out: track 0.00 -> 15.1 mm
- net GND: track 50.8 -> 36.5 mm, vias 10 -> 9
- net /OutputAmplifier/G0: track 13.9 -> 0.00 mm
- net /OutputAmplifier/G0_out: track 0.00 -> 12.8 mm
- net /OutputAmplifier/G1: track 11.9 -> 0.00 mm
- net /Band Pass Filter/F1_Out: track 28.2 -> 17.4 mm, vias 0 -> 1
- net VCC: track 40.7 -> 30.0 mm
- net /OutputAmplifier/G2: track 9.83 -> 0.00 mm
- net AGND: track 26.7 -> 35.2 mm
- net Net-(U4-CLK): track 12.9 -> 20.0 mm
- net Net-(J2-Pad1): track 15.1 -> 19.4 mm
- net /Band Pass Filter/F3_Out: track 22.7 -> 19.4 mm
- net Net-(U4-~{CS}): track 26.4 -> 23.4 mm
- net /Band Pass Filter/F2_Out: track 8.01 -> 9.37 mm
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Other:
- board size 25.6 x 52.2 mm -> 25.4 x 44.1 mm
- board text removed: "+"
- board text removed: "-"
- board text removed: "0"
- board text removed: "1"
- board text removed: "2 1 0"
- board text removed: "A"
- board text removed: "CLK"
- board text removed: "CS"
- board text removed: "DOUT"

Commit message: Fixed routing
Parts:
- moved ? 2.65 mm to (144.8, 111.3)
Routing:
- net /OutputAmplifier/Amp_Out: track 16.7 -> 13.1 mm

Commit message: Hopefully it works this time
Parts:
- moved R25 0.56 mm to (159.6, 87.5)
- moved D1 0.51 mm to (159.6, 84.8)
Changed lines of the file:
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@@
     (property "Sheetname" "Band Pass Filter")
     (property "ki_description" "RES SMD 698 OHM 1% 1/10W 0603")
-    (fp_text reference "R10" (at -0.87681 0.72561 unlocked) (layer "F.SilkS")
+    (fp_text reference "R10" (at -0.87681 1.23361 unlocked) (layer "F.SilkS")
         (effects (font (size 0.635 0.762) (thickness 0.127)) (justify left bottom))
     )
@@
   )
   (footprint "AltiumImports:SMD-0603-RES" (layer "F.Cu")
-    (at 160.10821 87.544675)
+    (at 159.55006 87.539005)
     (property "Part Number" "ERJ-3EKF3000V")
     (property "Sheetfile" "AcousticsSingleChannel.kicad_sch")
@@
   )
   (footprint "AltiumImports:VISH-TLMX1100_V" (layer "F.Cu")
-    (at 160.05922 84.801345 90)
+    (at 159.55006 84.801345 90)
     (property "Part Number" "150080SS75000")
     (property "Sheetfile" "AcousticsSingleChannel.kicad_sch")
@@
     (style (thickness 0.254) (arrow_length 1.27) (text_position_mode 0) (extension_height 0.58642) (extension_offset 0) keep_text_aligned)
   )
-  (segment (start 159.80406 89.965005) (end 160.19394 89.575125) (width 0.254) (layer "F.Cu") (net 1))
   (segment (start 149.5841 115.889745) (end 152.1423 115.889745) (width 0.254) (layer "F.Cu") (net 1))
   (segment (start 143.50033 106.893845) (end 145.48631 106.893845) (width 0.254) (layer "F.Cu") (net 1))
@@
   (segment (start 145.48631 106.893845) (end 147.12533 106.893845) (width 0.254) (layer "F.Cu") (net 1))
   (segment (start 154.72406 96.442005) (end 155.10006 96.442005) (width 0.127) (layer "F.Cu") (net 1))
-  (segment (start 152.36483 117.284755) (end 152.36483 116.145625) (width 0.254) (layer "F.Cu") (net 1))
-  (segment (start 160.19394 89.575125) (end 160.19394 88.442045) (width 0.254) (layer "F.Cu") (net 1))
   (segment (start 139.86274 117.164605) (end 139.7598 117.061665) (width 0.127) (layer "F.Cu") (net 1))
   (segment (start 147.12533 106.893845) (end 147.78082 107.549335) (width 0.254) (layer "F.Cu") (net 1))
@@
   (segment (start 137.84737 116.045705) (end 138.12167 115.771405) (width 0.254) (layer "F.Cu") (net 1))
   (segment (start 152.02749 91.369195) (end 152.02749 89.603575) (width 0.254) (layer "F.Cu") (net 1))
+  (segment (start 159.55006 89.965005) (end 159.55006 88.314005) (width 0.127) (layer "F.Cu") (net 1))
   (segment (start 137.84737 117.024085) (end 137.84737 116.045705) (width 0.254) (layer "F.Cu") (net 1))
   (segment (start 141.38906 117.164605) (end 139.86274 117.164605) (width 0.254) (layer "F.Cu") (net 1))
@@
   (segment (start 139.72222 116.045705) (end 139.72222 117.024085) (width 0.254) (layer "F.Cu") (net 1))
   (segment (start 154.97806 105.993005) (end 154.97806 107.364005) (width 0.254) (layer "F.Cu") (net 1))
+  (segment (start 152.36483 117.016005) (end 152.36483 116.145625) (width 0.127) (layer "F.Cu") (net 1))
   (segment (start 136.8842 107.971435) (end 136.8842 106.518795) (width 0.254) (layer "F.Cu") (net 1))
+  (segment (start 152.36483 116.145625) (end 152.38151 116.128945) (width 0.127) (layer "F.Cu") (net 1))
   (segment (start 138.76724 107.771025) (end 138.76724 105.543095) (width 0.254) (layer "F.Cu") (net 1))
   (via (at 138.76724 105.543095) (size 0.55) (drill 0.2) (layers "F.Cu" "B.Cu") (net 1))
-  (via (at 159.80406 89.965005) (size 0.55) (drill 0.2) (layers "F.Cu" "B.Cu") (net 1))
+  (via (at 159.55006 89.965005) (size 0.55) (drill 0.2) (layers "F.Cu" "B.Cu") (net 1))
   (via (at 141.38906 117.164605) (size 0.762) (drill 0.3556) (layers "F.Cu" "B.Cu") (net 1))
   (via (at 154.97806 107.364005) (size 0.55) (drill 0.2) (layers "F.Cu" "B.Cu") (net 1))
   (via (at 151.64403 87.656185) (size 0.55) (drill 0.2) (layers "F.Cu" "B.Cu") (net 1))
   (via (at 147.80131 107.528845) (size 0.55) (drill 0.2) (layers "F.Cu" "B.Cu") (net 1))
-  (via (at 152.36483 117.284755) (size 0.55) (drill 0.2) (layers "F.Cu" "B.Cu") (net 1))
+  (via (at 152.36483 117.016005) (size 0.55) (drill 0.2) (layers "F.Cu" "B.Cu") (net 1))
   (segment (start 140.75297 106.886465) (end 141.94296 106.886465) (width 0.254) (layer "F.Cu") (net 2))
   (segment (start 152.02749 85.064945) (end 152.02749 83.703575) (width 0.254) (layer "F.Cu") (net 2))
@@
   (segment (start 149.16742 107.552225) (end 149.8258 106.893845) (width 0.254) (layer "F.Cu") (net 2))
   (segment (start 137.8098 112.714335) (end 137.8098 110.465765) (width 0.254) (layer "F.Cu") (net 2))
-  (segment (start 160.04697 84.047425) (end 160.04697 82.498885) (width 0.254) (layer "F.Cu") (net 2))
   (segment (start 137.8098 110.465765) (end 137.8098 110.302625) (width 0.254) (layer "F.Cu") (net 2))
   (segment (start 151.93516 94.228435) (end 151.93516 93.313965) (width 0.254) (layer "F.Cu") (net 2))
   (segment (start 137.8098 112.741965) (end 138.4598 112.741965) (width 0.254) (layer "F.Cu") (net 2))
   (segment (start 137.8098 110.302625) (end 138.5499 109.562515) (width 0.254) (layer "F.Cu") (net 2))
+  (segment (start 159.55006 82.599005) (end 159.55006 84.076345) (width 0.127) (layer "F.Cu") (net 2))
   (segment (start 141.42467 85.460765) (end 143.14325 87.179345) (width 0.254) (layer "F.Cu") (net 2))
   (segment (start 145.79595 117.844975) (end 147.15669 117.844975) (width 0.254) (layer "F.Cu") (net 2))
@@
   (via (at 153.52592 114.393665) (size 0.55) (drill 0.2) (layers "F.Cu" "B.Cu") (net 2))
   (via (at 140.75406 106.881405) (size 0.55) (drill 0.2) (layers "F.Cu" "B.Cu") (net 2))
-  (via (at 160.04697 82.498885) (size 0.55) (drill 0.2) (layers "F.Cu" "B.Cu") (net 2))
+  (via (at 159.55006 82.599005) (size 0.55) (drill 0.2) (layers "F.Cu" "B.Cu") (net 2))
   (via (at 143.94993 119.125595) (size 0.55) (drill 0.2) (layers "F.Cu" "B.Cu") (net 2))
   (segment (start 151.37749 83.703575) (end 151.37749 82.472675) (width 0.254) (layer "F.Cu") (net 3))
@@
   (via (at 152.05706 97.077005) (size 0.55) (drill 0.2) (layers "F.Cu" "B.Cu") (net 3))
   (via (at 158.56849 89.270005) (size 0.55) (drill 0.2) (layers "F.Cu" "B.Cu") (net 3))
-  (segment (start 160.10045 86.798565) (end 160.10045 85.670885) (width 0.254) (layer "F.Cu") (net 4))
+  (segment (start 159.55006 85.526345) (end 159.55006 86.764005) (width 0.127) (layer "F.Cu") (net 4))
   (segment (start 142.40506 120.699005) (end 141.51606 119.810005) (width 0.254) (layer "F.Cu") (net 5))
   (segment (start 139.23006 118.921005) (end 140.62706 118.921005) (width 0.254) (layer "F.Cu") (net 5))
