File: AcousticsSingleChannel.kicad_pcb (KiCad board)
At the start: 4 copper layers, 25.4 x 25.4 mm, 35 parts, among them J1 Conn_01x04_Pin, J2 Conn_01x04_Pin, J4 Conn_01x09_Pin, U1 OPA1604AIPWR, U2 ADS127L21IRUKT, U3 LTC6910-3CTS8#TRPBF

Commit message: tracks
Parts:
- moved C4 0.46 mm to (138.3, 99.1)
Routing:
- net /RESET: track 23.8 -> 24.7 mm
Changed lines of the file:
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@@
 	(footprint "AltiumImports:SMD-0603C"
 		(layer "B.Cu")
-		(at 138.72206 98.855005 180)
+		(at 138.34106 99.109005 180)
 		(property "Reference" "C4"
 			(at 0.762 -0.635 0)
@@
 	)
 	(segment
-		(start 143.900359 91.743005)
-		(end 142.56106 91.743005)
-		(width 0.127)
+		(start 151.07106 92.378005)
+		(end 153.32706 92.378005)
+		(width 0.254)
 		(layer "F.Cu")
 		(net 1)
 	)
 	(segment
-		(start 143.92906 91.714304)
-		(end 143.900359 91.743005)
-		(width 0.127)
+		(start 143.900359 91.743005)
+		(end 143.92906 91.714304)
+		(width 0.254)
 		(layer "F.Cu")
 		(net 1)
 	)
 	(segment
-		(start 151.11798 92.424925)
-		(end 151.07106 92.378005)
+		(start 153.32706 92.378005)
+		(end 153.58106 92.632005)
 		(width 0.254)
 		(layer "F.Cu")
@@
 	)
 	(segment
-		(start 153.32706 92.378005)
+		(start 151.11798 92.424925)
 		(end 151.07106 92.378005)
-		(width 0.127)
+		(width 0.254)
 		(layer "F.Cu")
 		(net 1)
 	)
 	(segment
-		(start 153.58106 92.632005)
-		(end 153.32706 92.378005)
-		(width 0.127)
+		(start 142.56106 91.743005)
+		(end 143.900359 91.743005)
+		(width 0.254)
 		(layer "F.Cu")
 		(net 1)
@@
 	)
 	(segment
-		(start 138.72206 99.630005)
-		(end 139.48406 98.868005)
-		(width 0.127)
-		(layer "B.Cu")
-		(net 1)
-	)
-	(segment
 		(start 140.31056 91.916504)
 		(end 141.97456 91.916504)
@@
 	)
 	(segment
-		(start 139.48406 97.450006)
-		(end 139.615861 97.318205)
-		(width 0.127)
-		(layer "B.Cu")
-		(net 1)
-	)
-	(segment
 		(start 141.97456 91.916504)
 		(end 143.30706 90.584004)
@@
 	)
 	(segment
+		(start 138.70906 99.884005)
+		(end 139.23006 99.363005)
+		(width 0.254)
+		(layer "B.Cu")
+		(net 1)
+	)
+	(segment
 		(start 139.615861 93.589205)
 		(end 139.615861 92.611203)
@@
 	)
 	(segment
-		(start 136.452061 95.537004)
-		(end 135.16606 96.823005)
-		(width 0.127)
+		(start 139.23006 97.825807)
+		(end 139.615861 97.440006)
+		(width 0.254)
 		(layer "B.Cu")
 		(net 1)
 	)
 	(segment
-		(start 139.615861 97.318205)
+		(start 138.46806 95.537004)
+		(end 136.198061 95.537004)
+		(width 0.254)
+		(layer "B.Cu")
+		(net 1)
+	)
+	(segment
+		(start 139.615861 97.440006)
 		(end 139.615861 96.684805)
-		(width 0.127)
+		(width 0.254)
 		(layer "B.Cu")
 		(net 1)
 	)
 	(segment
-		(start 139.48406 98.868005)
-		(end 139.48406 97.450006)
-		(width 0.127)
+		(start 136.198061 95.537004)
+		(end 135.29306 96.442005)
+		(width 0.254)
 		(layer "B.Cu")
 		(net 1)
 	)
 	(segment
-		(start 138.46806 95.537004)
-		(end 136.452061 95.537004)
-		(width 0.127)
+		(start 138.34106 99.884005)
+		(end 138.70906 99.884005)
+		(width 0.254)
+		(layer "B.Cu")
+		(net 1)
+	)
+	(segment
+		(start 139.23006 99.363005)
+		(end 139.23006 97.825807)
+		(width 0.254)
 		(layer "B.Cu")
 		(net 1)
@@
 	)
 	(segment
-		(start 134.97306 95.137005)
-		(end 134.55706 95.553005)
-		(width 0.127)
+		(start 138.46806 95.137005)
+		(end 134.97306 95.137005)
+		(width 0.254)
 		(layer "B.Cu")
 		(net 6)
 	)
 	(segment
-		(start 138.46806 95.137005)
-		(end 134.97306 95.137005)
-		(width 0.127)
+		(start 134.97306 95.137005)
+		(end 134.55706 95.553005)
+		(width 0.254)
 		(layer "B.Cu")
 		(net 6)
 	)
 	(segment
-		(start 139.215859 96.684805)
-		(end 139.215859 97.586206)
-		(width 0.127)
+		(start 138.34106 97.559604)
+		(end 139.215859 96.684805)
+		(width 0.254)
 		(layer "B.Cu")
 		(net 7)
 	)
 	(segment
-		(start 139.215859 97.586206)
-		(end 138.72206 98.080005)
-		(width 0.127)
+		(start 138.34106 98.334005)
+		(end 138.34106 97.559604)
+		(width 0.254)
 		(layer "B.Cu")
 		(net 7)
@@
 		(start 143.659059 95.537004)
 		(end 144.56406 96.442005)
-		(width 0.127)
+		(width 0.254)
 		(layer "B.Cu")
 		(net 10)
@@
 		(start 141.56366 95.537004)
 		(end 143.659059 95.537004)
-		(width 0.127)
+		(width 0.254)
 		(layer "B.Cu")
 		(net 10)
@@
 		(start 141.56366 94.737006)
 		(end 145.526061 94.737006)
-		(width 0.127)
+		(width 0.254)
 		(layer "B.Cu")
 		(net 11)
@@
 		(start 145.526061 94.737006)
 		(end 146.85006 96.061005)
-		(width 0.127)
+		(width 0.254)
 		(layer "B.Cu")
 		(net 11)
@@
 	)
 	(segment
-		(start 144.81806 95.299005)
-		(end 144.65606 95.137005)
-		(width 0.127)
-		(layer "B.Cu")
-		(net 13)
-	)
-	(segment
-		(start 144.65606 95.137005)
-		(end 141.56366 95.137005)
-		(width 0.127)
+		(start 145.16406 95.137005)
+		(end 145.32606 95.299005)
+		(width 0.254)
 		(layer "B.Cu")
 		(net 13)
 	)
 	(segment
-		(start 145.32606 95.299005)
-		(end 144.81806 95.299005)
-		(width 0.127)
+		(start 141.56366 95.137005)
+		(end 145.16406 95.137005)
+		(width 0.254)
 		(layer "B.Cu")
 		(net 13)
@@
 	(segment
 		(start 141.56366 94.337004)
-		(end 146.396059 94.337004)
-		(width 0.127)
+		(end 141.56366 94.108405)
+		(width 0.254)
 		(layer "B.Cu")
 		(net 17)
 	)
 	(segment
-		(start 146.396059 94.337004)
+		(start 145.45306 93.394005)
 		(end 147.86606 95.807005)
-		(width 0.127)
+		(width 0.254)
+		(layer "B.Cu")
+		(net 17)
+	)
+	(segment
+		(start 142.27806 93.394005)
+		(end 145.45306 93.394005)
+		(width 0.254)
+		(layer "B.Cu")
+		(net 17)
+	)
+	(segment
+		(start 141.56366 94.108405)
+		(end 142.27806 93.394005)
+		(width 0.254)
 		(layer "B.Cu")
 		(net 17)
@@
 	)
 	(segment
-		(start 140.01586 96.684805)
-		(end 140.01586 98.196205)
-		(width 0.127)
+		(start 140.01586 98.196205)
+		(end 139.99206 98.220005)
+		(width 0.254)
 		(layer "B.Cu")
 		(net 20)
@@
 	)
 	(segment
-		(start 140.01586 98.196205)
-		(end 139.99206 98.220005)
-		(width 0.127)
+		(start 140.01586 96.684805)
+		(end 140.01586 98.196205)
+		(width 0.254)
 		(layer "B.Cu")
 		(net 20)
@@
 	)
 	(segment
-		(start 142.281061 95.937006)
-		(end 141.56366 95.937006)
-		(width 0.127)
+		(start 141.56366 95.937006)
+		(end 142.281061 95.937006)
+		(width 0.254)
 		(layer "B.Cu")
 		(net 26)
 	)
 	(segment
-		(start 142.78606 96.442005)
-		(end 142.281061 95.937006)
-		(width 0.127)
+		(start 142.281061 95.937006)
+		(end 142.78606 96.442005)
+		(width 0.254)
 		(layer "B.Cu")
 		(net 26)
@@
 	)
 	(segment
-		(start 138.46806 94.737006)
-		(end 131.188061 94.737006)
-		(width 0.127)
+		(start 133.89606 87.422165)
+		(end 136.776088 87.422165)
+		(width 0.254)
 		(layer "B.Cu")
 		(net 29)
@@
 		(start 131.188061 94.737006)
 		(end 131.11506 94.664005)
-		(width 0.127)
+		(width 0.254)
 		(layer "B.Cu")
 		(net 29)
 	)
 	(segment
-		(start 133.89606 87.422165)
-		(end 136.776088 87.422165)
+		(start 138.46806 94.737006)
+		(end 131.188061 94.737006)
 		(width 0.254)
 		(layer "B.Cu")
@@
 	)
 	(segment
-		(start 145.07206 92.505005)
-		(end 149.13606 88.441005)
-		(width 0.127)
+		(start 131.11506 96.315005)
+		(end 131.11506 94.664005)
+		(width 0.254)
 		(layer "B.Cu")
 		(net 29)
 	)
 	(segment
-		(start 149.88506 89.190005)
-		(end 149.13606 88.441005)
-		(width 0.127)
+		(start 130.84806 92.571005)
+		(end 130.86406 92.587005)
+		(width 0.254)
 		(layer "B.Cu")
 		(net 29)
 	)
 	(segment
-		(start 130.84806 92.571005)
-		(end 130.86406 92.587005)
+		(start 149.88506 90.293005)
+		(end 149.88506 89.190005)
 		(width 0.254)
 		(layer "B.Cu")
@@
 	)
 	(segment
-		(start 140.866659 92.505005)
-		(end 145.07206 92.505005)
-		(width 0.127)
+		(start 131.11506 92.838005)
+		(end 130.86406 92.587005)
+		(width 0.254)
 		(layer "B.Cu")
 		(net 29)
@@
 	)
 	(segment
-		(start 131.11506 92.838005)
-		(end 130.86406 92.587005)
-		(width 0.127)
+		(start 149.88506 89.190005)
+		(end 149.13606 88.441005)
+		(width 0.254)
 		(layer "B.Cu")
 		(net 29)
 	)
 	(segment
-		(start 140.415859 93.589205)
-		(end 140.415859 92.955805)
-		(width 0.127)
+		(start 140.866659 92.378005)
+		(end 145.19906 92.378005)
+		(width 0.254)
 		(layer "B.Cu")
 		(net 29)
@@
 	(segment
 		(start 131.11506 94.664005)
-		(end 131.11506 96.315005)
-		(width 0.127)
+		(end 131.11506 92.838005)
+		(width 0.254)
 		(layer "B.Cu")
 		(net 29)
 	)
 	(segment
-		(start 140.415859 92.955805)
-		(end 140.866659 92.505005)
-		(width 0.127)
+		(start 140.415859 93.589205)
+		(end 140.415859 92.828805)
+		(width 0.254)
 		(layer "B.Cu")
 		(net 29)
 	)
 	(segment
-		(start 138.46806 94.337004)
-		(end 138.46806 94.737006)
-		(width 0.127)
+		(start 140.415859 92.828805)
+		(end 140.866659 92.378005)
+		(width 0.254)
 		(layer "B.Cu")
 		(net 29)
 	)
 	(segment
-		(start 131.11506 94.664005)
-		(end 131.11506 92.838005)
-		(width 0.127)
+		(start 145.19906 92.378005)
+		(end 149.13606 88.441005)
+		(width 0.254)
 		(layer "B.Cu")
 		(net 29)
 	)
 	(segment
-		(start 149.88506 90.293005)
-		(end 149.88506 89.190005)
-		(width 0.127)
+		(start 138.46806 94.337004)
+		(end 138.46806 94.737006)
+		(width 0.254)
 		(layer "B.Cu")
 		(net 29)

Commit message: tracks
Routing:
- net /RESET: track 24.7 -> 28.5 mm
Changed lines of the file:
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@@
 		(at 131.25806 88.269005)
 		(property "Reference" "R5"
-			(at 1.77408 0.61178 90)
+			(at -0.791 -1.479 0)
 			(unlocked yes)
 			(layer "F.SilkS")
@@
 		(at 132.02006 97.413005 180)
 		(property "Reference" "D2"
-			(at 1.27 -0.762 90)
+			(at 0.918 -1.95 0)
 			(unlocked yes)
 			(layer "F.SilkS")
@@
 		(at 131.25806 95.254005 180)
 		(property "Reference" "R21"
-			(at -1.778 -1.27 90)
+			(at -1.876 -1.061 90)
 			(unlocked yes)
 			(layer "F.SilkS")
@@
 		(at 150.09606 91.068005 90)
 		(property "Reference" "U3"
-			(at 1.357 1.707 0)
+			(at 0.976 1.58 0)
 			(unlocked yes)
 			(layer "F.SilkS")
@@
 		(at 134.57306 87.634005 -90)
 		(property "Reference" "C1"
-			(at 2.032 0.267 90)
+			(at -0.717 0.677 0)
 			(unlocked yes)
 			(layer "F.SilkS")
@@
 		(at 139.61106 91.743005)
 		(property "Reference" "U1"
-			(at -3.937 3.556 0)
+			(at 3.048 3.556 0)
 			(unlocked yes)
 			(layer "F.SilkS")
@@
 		(at 131.63906 92.587005 -90)
 		(property "Reference" "R25"
-			(at -0.93915 0.76933 0)
+			(at 1.188 1.553 90)
 			(unlocked yes)
 			(layer "F.SilkS")
@@
 		(at 151.93006 102.919005)
 		(property "Reference" "TP4"
-			(at -0.127 -2.413 0)
+			(at -3.556 -0.127 0)
 			(layer "F.SilkS")
 			(effects
@@
 		(at 141.54506 87.634005 90)
 		(property "Reference" "R2"
-			(at -0.762 -1.651 90)
+			(at 0.971 -0.791 0)
 			(unlocked yes)
 			(layer "F.SilkS")
@@
 		(at 137.74806 87.634005 90)
 		(property "Reference" "R4"
-			(at -2.159 -2.172 90)
+			(at 0.971 -0.804 0)
 			(unlocked yes)
 			(layer "F.SilkS")
@@
 		(at 145.70706 88.695005)
 		(property "Reference" "TP3"
-			(at 0.032 -2.4064 0)
+			(at -0.127 2.54 0)
 			(layer "F.SilkS")
 			(effects
@@
 		(at 134.56006 91.915005 90)
 		(property "Reference" "D1"
-			(at -0.799 -0.508 90)
+			(at -2.622 -0.664 0)
 			(unlocked yes)
 			(layer "F.SilkS")
@@
 		(at 152.05706 97.966005)
 		(property "Reference" "TP1"
-			(at -0.254 -2.413 0)
+			(at -3.175 0 0)
 			(layer "F.SilkS")
 			(effects
@@
 		(at 138.34106 99.109005 180)
 		(property "Reference" "C4"
-			(at 0.762 -0.635 0)
+			(at 0.889 -0.254 0)
 			(unlocked yes)
 			(layer "B.SilkS")
@@
 		(at 130.34006 96.315005 90)
 		(property "Reference" "C13"
-			(at -3.556 -0.127 270)
+			(at -2.286 0.889 0)
 			(unlocked yes)
 			(layer "B.SilkS")
@@
 		(at 149.88506 91.068005)
 		(property "Reference" "C12"
-			(at -1.778 1.143 270)
+			(at 0.648 2.834 0)
 			(unlocked yes)
 			(layer "B.SilkS")
@@
 		(at 142.53206 90.584004 90)
 		(property "Reference" "C5"
-			(at -1.667001 0.762 0)
+			(at -0.905001 3.556 0)
 			(unlocked yes)
 			(layer "B.SilkS")
@@
 		(tags "Through hole pin header THT 1x04 2.54mm single row")
 		(property "Reference" "J1"
-			(at -2.413 1.016 0)
+			(at -2.794 0.91186 0)
 			(layer "B.SilkS")
 			(effects
@@
 		(at 130.34006 94.664005 90)
 		(property "Reference" "C18"
-			(at -0.381 3.683 0)
+			(at -3.937 3.556 0)
 			(unlocked yes)
 			(layer "B.SilkS")
@@
 		(at 133.64206 102.792005 180)
 		(property "Reference" "R27"
-			(at -0.889 1.651 0)
+			(at 0.762 1.778 0)
 			(unlocked yes)
 			(layer "B.SilkS")
@@
 		(at 140.56356 100.709505)
 		(property "Reference" "C6"
-			(at 0.6985 2.3365 0)
+			(at 0.5715 2.7175 0)
 			(unlocked yes)
 			(layer "B.SilkS")
@@
 		(at 136.789088 88.184165)
 		(property "Reference" "C15"
-			(at 0.254 2.286 0)
+			(at 0.916972 2.54284 0)
 			(unlocked yes)
 			(layer "B.SilkS")
@@
 		(tags "Through hole pin header THT 1x09 2.54mm single row")
 		(property "Reference" "J4"
-			(at 3.23496 -21.43748 0)
+			(at 2.78384 -19.431 0)
 			(layer "B.SilkS")
 			(effects
@@
 		(at 133.89606 88.197165)
 		(property "Reference" "C14"
-			(at 1.016 2.286 0)
+			(at 0.762 2.40284 0)
 			(unlocked yes)
 			(layer "B.SilkS")
@@
 		(tags "Through hole pin header THT 1x04 2.54mm single row")
 		(property "Reference" "J2"
-			(at -2.413 -2.54254 0)
+			(at -2.54 -2.25044 0)
 			(layer "B.SilkS")
 			(effects
@@
 		(at 142.59556 102.106505)
 		(property "Reference" "C7"
-			(at 0.762 -1.3465 0)
+			(at 0.762 -1.8545 0)
 			(unlocked yes)
 			(layer "B.SilkS")
@@
 	)
 	(gr_text "BBA"
-		(at 148.24706 96.569005 0)
+		(at 151.04106 95.934005 0)
 		(layer "F.SilkS")
 		(effects
@@
 	)
 	(gr_text "SIG"
-		(at 144.56406 91.870005 0)
+		(at 144.56406 92.886005 0)
 		(layer "F.SilkS")
 		(effects
@@
 	)
 	(segment
-		(start 149.42562 106.094005)
+		(start 144.56406 97.712005)
 		(end 144.56406 101.232445)
 		(width 0.254)
@@
 	(segment
 		(start 144.56406 101.232445)
-		(end 144.56406 96.442005)
+		(end 149.42562 106.094005)
 		(width 0.254)
 		(layer "F.Cu")
@@
 	)
 	(via
-		(at 144.56406 96.442005)
+		(at 144.56406 97.712005)
 		(size 0.5334)
 		(drill 0.254)
@@
 	)
 	(segment
-		(start 143.659059 95.537004)
-		(end 144.56406 96.442005)
+		(start 141.56366 95.537004)
+		(end 143.532059 95.537004)
 		(width 0.254)
 		(layer "B.Cu")
@@
 	)
 	(segment
-		(start 141.56366 95.537004)
-		(end 143.659059 95.537004)
+		(start 143.532059 95.537004)
+		(end 144.56406 96.569005)
+		(width 0.254)
+		(layer "B.Cu")
+		(net 10)
+	)
+	(segment
+		(start 144.56406 96.569005)
+		(end 144.56406 97.712005)
 		(width 0.254)
 		(layer "B.Cu")
@@
 	)
 	(segment
-		(start 138.74492 101.372145)
-		(end 144.81806 95.299005)
+		(start 138.74492 106.094005)
+		(end 138.74492 102.007145)
 		(width 0.254)
 		(layer "F.Cu")
@@
 	)
 	(segment
-		(start 144.81806 95.299005)
+		(start 145.32606 95.426005)
 		(end 145.32606 95.299005)
 		(width 0.254)
@@
 	)
 	(segment
-		(start 138.74492 106.094005)
-		(end 138.74492 101.372145)
+		(start 138.74492 102.007145)
+		(end 145.32606 95.426005)
 		(width 0.254)
 		(layer "F.Cu")
@@
 	)
 	(segment
-		(start 146.72306 95.172005)
-		(end 147.61206 95.172005)
+		(start 147.86606 95.807005)
+		(end 146.08806 94.029005)
 		(width 0.254)
 		(layer "In1.Cu")
@@
 	)
 	(segment
-		(start 136.20492 105.690145)
-		(end 146.72306 95.172005)
+		(start 141.38906 100.909865)
+		(end 136.20492 106.094005)
 		(width 0.254)
 		(layer "In1.Cu")
@@
 	)
 	(segment
-		(start 147.61206 95.172005)
-		(end 147.86606 95.426005)
+		(start 136.20492 106.094005)
+		(end 136.20492 105.690145)
 		(width 0.254)
 		(layer "In1.Cu")
@@
 	)
 	(segment
-		(start 136.20492 106.094005)
-		(end 136.20492 105.690145)
+		(start 143.29406 94.029005)
+		(end 141.38906 95.934005)
 		(width 0.254)
 		(layer "In1.Cu")
@@
 	)
 	(segment
-		(start 147.86606 95.426005)
-		(end 147.86606 95.807005)
+		(start 141.38906 95.934005)
+		(end 141.38906 100.909865)
+		(width 0.254)
+		(layer "In1.Cu")
+		(net 17)
+	)
+	(segment
+		(start 146.08806 94.029005)
+		(end 143.29406 94.029005)
 		(width 0.254)
 		(layer "In1.Cu")
