File: Band Pass Filter.kicad_sch (KiCad schematic)
At the start: 23 parts, among them U1 OPA1604AIPWR, U2 OPA1604AIPWR

Commit message: Fix various net and footprint issues
Connections:
- net BPF IN renamed BPF_IN
- net BPF OUT renamed BPF_OUT

Commit message: Cleanup symbol table
Parts:
- C10, C3, C4, C5, C6, C7, C8, C9: ALTIUM_VALUE 1000pF -> (none); DATASHEET LINK https://www.digikey.com/en/products/detail/walsin-technolog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 -> (none); MANUFACTURER Walsin Technology Corporation -> (none); MANUFACTURER PART NUMBER 0603N102F500CT -> (none); OPERATING TEMPERATURE -55°C ~ 125°C -> (none); PACKAGE / CASE 0603 (1608 Metric) -> (none); Part Number (none) -> 0603N102F500CT
- C17: ALTIUM_VALUE 1µF -> (none); DATASHEET LINK https://www.digikey.com/en/products/detail/samsung-electro-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 -> (none); MANUFACTURER Samsung Electro-Mechanics -> (none); MANUFACTURER PART NUMBER CL10A105KA8NNNC -> (none); OPERATING TEMPERATURE -55°C ~ 125°C -> (none); PACKAGE / CASE 0603 (1608 Metric) -> (none); Part Number (none) -> CL10A105KA8NNNC
- R10: ALTIUM_VALUE 698 -> (none); DATASHEET LINK https://www.digikey.com/en/products/detail/panasonic-electr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 -> (none); MANUFACTURER Panasonic Electronic Components -> (none); MANUFACTURER PART NUMBER ERJ-3EKF6980V -> (none); OPERATING TEMPERATURE -55°C ~ 155°C -> (none); PACKAGE / CASE 0603 (1608 Metric) -> (none); Part Number (none) -> ERJ-3EKF6980V
- R11: ALTIUM_VALUE 536 -> (none); DATASHEET LINK https://www.digikey.com/en/products/detail/panasonic-electr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 -> (none); MANUFACTURER Panasonic Electronic Components -> (none); MANUFACTURER PART NUMBER ERJ-3EKF5360V -> (none); OPERATING TEMPERATURE -55°C ~ 155°C -> (none); PACKAGE / CASE 0603 (1608 Metric) -> (none); Part Number (none) -> ERJ-3EKF5360V
- R12: ALTIUM_VALUE 165k -> (none); DATASHEET LINK https://www.digikey.com/en/products/detail/panasonic-electr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 -> (none); MANUFACTURER Panasonic Electronic Components -> (none); MANUFACTURER PART NUMBER ERJ-3EKF1653V -> (none); OPERATING TEMPERATURE -55°C ~ 155°C -> (none); PACKAGE / CASE 0603 (1608 Metric) -> (none); Part Number (none) -> ERJ-3EKF1653V
- R13: ALTIUM_VALUE 86.6k -> (none); DATASHEET LINK https://www.digikey.com/en/products/detail/panasonic-electr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 -> (none); MANUFACTURER Panasonic Electronic Components -> (none); MANUFACTURER PART NUMBER ERJ-3EKF8662V -> (none); OPERATING TEMPERATURE -55°C ~ 155°C -> (none); PACKAGE / CASE 0603 (1608 Metric) -> (none); Part Number (none) -> ERJ-3EKF8662V
- R14: ALTIUM_VALUE 11k -> (none); DATASHEET LINK https://www.digikey.com/en/products/detail/panasonic-electr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 -> (none); MANUFACTURER Panasonic Electronic Components -> (none); MANUFACTURER PART NUMBER ERJ-3EKF1102V -> (none); OPERATING TEMPERATURE -55°C ~ 155°C -> (none); PACKAGE / CASE 0603 (1608 Metric) -> (none); Part Number (none) -> ERJ-3EKF1102V
- R15: ALTIUM_VALUE 5.76k -> (none); DATASHEET LINK https://www.digikey.com/en/products/detail/panasonic-electr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 -> (none); MANUFACTURER Panasonic Electronic Components -> (none); MANUFACTURER PART NUMBER ERJ-3EKF5761V -> (none); OPERATING TEMPERATURE -55°C ~ 155°C -> (none); PACKAGE / CASE 0603 (1608 Metric) -> (none); Part Number (none) -> ERJ-3EKF5761V
- R16: ALTIUM_VALUE 332 -> (none); DATASHEET LINK https://www.digikey.com/en/products/detail/panasonic-electr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 -> (none); MANUFACTURER Panasonic Electronic Components -> (none); MANUFACTURER PART NUMBER ERJ-3EKF3320V -> (none); OPERATING TEMPERATURE -55°C ~ 155°C -> (none); PACKAGE / CASE 0603 (1608 Metric) -> (none); Part Number (none) -> ERJ-3EKF3320V
- R17: ALTIUM_VALUE 174 -> (none); DATASHEET LINK https://www.digikey.com/en/products/detail/panasonic-electr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 -> (none); MANUFACTURER Panasonic Electronic Components -> (none); MANUFACTURER PART NUMBER ERJ-3EKF1740V -> (none); OPERATING TEMPERATURE -55°C ~ 155°C -> (none); PACKAGE / CASE 0603 (1608 Metric) -> (none); Part Number (none) -> ERJ-3EKF1740V
- R6: ALTIUM_VALUE 54.9k -> (none); DATASHEET LINK https://www.digikey.com/en/products/detail/panasonic-electr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 -> (none); MANUFACTURER Panasonic Electronic Components -> (none); MANUFACTURER PART NUMBER ERJ-3EKF5492V -> (none); OPERATING TEMPERATURE -55°C ~ 155°C -> (none); PACKAGE / CASE 0603 (1608 Metric) -> (none); Part Number (none) -> ERJ-3EKF5492V
- R7: ALTIUM_VALUE 41.2k -> (none); DATASHEET LINK https://www.digikey.com/en/products/detail/yageo/RC0603FR-0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 -> (none); MANUFACTURER Panasonic Electronic Components -> (none); MANUFACTURER PART NUMBER ERJ-3EKF4122V -> (none); OPERATING TEMPERATURE -55°C ~ 155°C -> (none); PACKAGE / CASE 0603 (1608 Metric) -> (none); Part Number (none) -> ERJ-3EKF4122V
- R8: ALTIUM_VALUE 17.4k -> (none); DATASHEET LINK https://www.digikey.com/en/products/detail/panasonic-electr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 -> (none); MANUFACTURER Panasonic Electronic Components -> (none); MANUFACTURER PART NUMBER ERJ-3EKF1742V -> (none); OPERATING TEMPERATURE -55°C ~ 155°C -> (none); PACKAGE / CASE 0603 (1608 Metric) -> (none); Part Number (none) -> ERJ-3EKF1742V
- R9: ALTIUM_VALUE 13k -> (none); DATASHEET LINK https://www.digikey.com/en/products/detail/panasonic-electr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 -> (none); MANUFACTURER Panasonic Electronic Components -> (none); MANUFACTURER PART NUMBER ERJ-3EKF1302V -> (none); OPERATING TEMPERATURE -55°C ~ 155°C -> (none); PACKAGE / CASE 0603 (1608 Metric) -> (none); Part Number (none) -> ERJ-3EKF1302V
- U1, U2: DATASHEET LINK https://www.digikey.com/en/products/detail/texas-instrument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 -> (none); MANUFACTURER Texas Instruments -> (none); MANUFACTURER PART NUMBER OPA1604AIPWR -> (none); OPERATING TEMPERATURE -40°C ~ 85°C -> (none); PACKAGE / CASE 14-TSSOP -> (none); Part Number (none) -> OPA1604AIPWR

Commit message: Ready for review
Connections:
- net VCC renamed +3.3V
Other:
- note removed: "${##}"
- note removed: "${#}"
- note removed: "${ADDRESS1}"
- note removed: "${ADDRESS2}"
- note removed: "${ADDRESS3}"
- note removed: "${ADDRESS4}"
- note removed: "${CAGE_CODE}"
- note removed: "${DOC_NO_ASSY_DWG}"
- note removed: "${DOC_NO_BOM}"
- note removed: "${DOC_NO_FAB_DWG}"
- note removed: "${DOC_NO_SCH_DWG}"
- note removed: "${FILENAME}"
- note removed: "${ITEMREVISION}"
- note removed: "${ITEM}"
- note removed: "${PCB_DWG_NO}"
- note removed: "${PROJECT}"
- note removed: "${SCH_SCALE}"
- note removed: "${TITLE}"
- note removed: "${VERSIONCONTROL_PROJFOLDERREVNUMBER}"
- note removed: "${VERSIONCONTROL_REVNUMBER}"
- note removed: "APPROVED"
- note removed: "B"
- note removed: "CAGE CODE"
- note removed: "DATE"
- note removed: "DESCRIPTION"
- note removed: "DESIGN ITEM:"
- note removed: "DOCUMENT REVISION:"
- note removed: "DWG NO."
- note removed: "DWG. NO."
- note removed: "FILE NAME"
- note removed: "OF"
- note removed: "PROJECT"
- note removed: "PROJECT REVISION:"
- note removed: "REFERENCE DOCUMENTS"
- note removed: "REV"
- note removed: "REV."
- note removed: "REVISION"
- note removed: "SCALE:"
- note removed: "SHEET"
- note removed: "SHT."
- note removed: "SIZE"
- note removed: "TITLE"
- moved on the sheet: C17, C9, R14, R15, R16
