File: BufferBiasAmp.kicad_sch (KiCad schematic)
At the start: 12 parts, among them SW2 Switch_Omron_A6S-1104-PH_eec, U1 OPA1604AIPWR

Commit message: Fix various net and footprint issues
Connections:
- net BBA IN renamed BBA_IN
- net BBA OUT renamed BBA_OUT
Changed lines of the file:
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@@
     (effects (font (size 1.27 1.27)) (justify left bottom))
   )
-  (label "BUF_IN" (at 53.34 114.3 0)
+  (label "BUF_IN" (at 53.34 114.3 0) (fields_autoplaced)
     (effects (font (size 1.27 1.27)) (justify left bottom))
   )
-  (label "BBAmp_IN" (at 146.05 111.76 0)
+  (label "BBAmp_IN" (at 146.05 111.76 0) (fields_autoplaced)
     (effects (font (size 1.27 1.27)) (justify left bottom))
   )
-  (label "BIAS_IN" (at 87.63 109.22 0)
+  (label "BIAS_IN" (at 87.63 109.22 0) (fields_autoplaced)
     (effects (font (size 1.27 1.27)) (justify left bottom))
   )
-  (label "BIAS_OUT" (at 127 88.9 0)
+  (label "BIAS_OUT" (at 127 88.9 0) (fields_autoplaced)
     (effects (font (size 1.27 1.27)) (justify left bottom))
   )
-  (label "BUF_OUT" (at 69.85 88.9 0)
+  (label "BUF_OUT" (at 69.85 88.9 0) (fields_autoplaced)
     (effects (font (size 1.27 1.27)) (justify left bottom))
   )
-  (label "BBA_OUT" (at 184.15 109.22 0)
+  (label "BBA_OUT" (at 184.15 109.22 0) (fields_autoplaced)
     (effects (font (size 1.27 1.27)) (justify left bottom))
   )
-  (hierarchical_label "BBA OUT" (shape output) (at 196.85 109.22 0) (fields_autoplaced)
+  (hierarchical_label "BBA_OUT" (shape output) (at 196.85 109.22 0) (fields_autoplaced)
     (effects (font (size 1.27 1.27)) (justify left))
   )
-  (hierarchical_label "BBA IN" (shape input) (at 31.75 123.19 180) (fields_autoplaced)
+  (hierarchical_label "BBA_IN" (shape input) (at 31.75 123.19 180) (fields_autoplaced)
     (effects (font (size 1.27 1.27)) (justify right))
   )

Commit message: Cleanup symbol table
Parts:
- C1: ALTIUM_VALUE 5100pF -> (none); DATASHEET LINK https://www.digikey.com/en/products/detail/murata-electroni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 -> (none); MANUFACTURER Murata Electronics North America -> (none); MANUFACTURER PART NUMBER GRM1887U1H512JA01D -> (none); OPERATING TEMPERATURE -55°C ~ 125°C -> (none); PACKAGE / CASE 0603 (1608 Metric) -> (none); Part Number (none) -> GRM1887U1H512JA01D
- C16: ALTIUM_VALUE 1µF -> (none); DATASHEET LINK https://www.digikey.com/en/products/detail/samsung-electro-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 -> (none); MANUFACTURER Samsung Electro-Mechanics -> (none); MANUFACTURER PART NUMBER CL10A105KA8NNNC -> (none); OPERATING TEMPERATURE -55°C ~ 125°C -> (none); PACKAGE / CASE 0603 (1608 Metric) -> (none); Part Number (none) -> CL10A105KA8NNNC
- C2: @ QTY 0 -> (none); ALTIUM_VALUE 5100pF -> (none); APPLICATIONS General Purpose -> (none); DATASHEETS http://www.murata.com/~/media/webrenewal/support/library/ca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 -> (none); DIGI-KEY PART NUMBER 490-6399-1-ND -> (none); FACTORY STOCK 0 -> (none); FEATURES - -> (none); HEIGHT - SEATED (MAX) - -> (none); IMAGE //media.digikey.com/Renders/Murata%20Renders/ZRB-SERIES-040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 -> (none); LEAD SPACING - -> (none); LEAD STYLE - -> (none); MANUFACTURER Murata Electronics North America -> (none); MINIMUM QUANTITY 1 -> (none); MOUNTING TYPE Surface Mount, MLCC -> (none); OPERATING TEMPERATURE -55°C ~ 125°C -> (none); PACKAGE / CASE 0603 (1608 Metric) -> (none); PACKAGING Cut Tape (CT) -> (none); PART NUMBER GRM1887U1H512JA01D -> (none); PART STATUS Active -> (none); Part Number (none) -> GRM1887U1H512JA01D; QUANTITY AVAILABLE 12288 -> (none); RATINGS - -> (none); SERIES GRM -> (none); SIZE / DIMENSION 0.063" L x 0.031" W (1.60mm x 0.80mm) -> (none); TEMPERATURE COEFFICIENT U2J -> (none); THICKNESS (MAX) 0.035" (0.90mm) -> (none); TOLERANCE ±5% -> (none); UNIT PRICE (USD) 0.2 -> (none); VOLTAGE 50V -> (none)
- D2: AMBIENT TEMPERATURE RANGE HIGH +100°C -> (none); AMBIENT TEMPERATURE RANGE LOW -40°C -> (none); AUTOMOTIVE Yes -> (none); AUTOMOTIVE GRADE Grade 3 -> (none); CATEGORY Diode -> (none); COLOUR Pure green -> (none); COMPONENTLINK2DESCRIPTION Datasheet -> (none); COMPONENTLINK2URL http://www.vishay.com/docs/83173/tlmb1100.pdf -> (none); DESCRIPTION Green 561nm LED Indication - Discrete 2.1V 0603 (1608 Metri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 -> (none); DEVICE CLASS L1 Optoelectronics -> (none); DEVICE CLASS L2 LEDs -> (none); DEVICE CLASS L3 unset -> (none); DIGIKEY DESCRIPTION LED GREEN 0603 SMD -> (none); FORWARD CURRENT 20mA -> (none); FORWARD VOLTAGE 2.1V -> (none); HEIGHT 0.65mm -> (none); LEAD FREE Yes -> (none); LED ORIENTATION Top View -> (none); LUMINOUS INTENSITY 15mcd -> (none); MANUFACTURER Vishay -> (none); MANUFACTURER PART NUMBER TLMP1100-GS08 -> (none); MAX JUNCTION TEMP +120°C -> (none); MOUSER DESCRIPTION Standard LEDs - SMD Pure Green -> (none); OCTOPART https://octopart.com/tlmp1100-gs08-vishay-55433993 -> (none); PACKAGE 6.541-5056.01-4 -> (none); PEAK EMMISION WAVELENGTH 562nm -> (none); POWER DISSIPATION 90mW -> (none); Part Number (none) -> TLMP1100-GS08; REVERSE VOLTAGE 6V -> (none); ROHS TRUE -> (none); TEMPERATURE to +120°C -> (none); TEMPERATURE RANGE HIGH +120°C -> (none); VIEWING ANGLE 160° -> (none); WAVELENGTH 561nm -> (none)
- R1, R2, R4: ALTIUM_VALUE 10k -> (none); DATASHEET LINK https://www.digikey.com/en/products/detail/stackpole-electr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 -> (none); MANUFACTURER Panasonic Electronic Components -> (none); MANUFACTURER PART NUMBER RNCP0603FTD10K0 -> (none); OPERATING TEMPERATURE -55°C ~ 155°C -> (none); PACKAGE / CASE 0603 (1608 Metric) -> (none); Part Number (none) -> RNCP0603FTD10K0
- R21: ALTIUM_VALUE 300 -> (none); DATASHEET LINK https://www.digikey.com/en/products/detail/panasonic-electr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 -> (none); MANUFACTURER Panasonic Electronic Components -> (none); MANUFACTURER PART NUMBER ERJ-3EKF3000V -> (none); OPERATING TEMPERATURE -55°C ~ 155°C -> (none); PACKAGE / CASE 0603 (1608 Metric) -> (none); Part Number (none) -> ERJ-3EKF3000V
- R3: ALTIUM_VALUE 1k -> (none); DATASHEET LINK https://www.digikey.com/en/products/detail/stackpole-electr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 -> (none); MANUFACTURER Stackpole Electronics Inc -> (none); MANUFACTURER PART NUMBER RNCP0603FTD1K00 -> (none); OPERATING TEMPERATURE -55°C ~ 155°C -> (none); PACKAGE / CASE 0603 (1608 Metric) -> (none); Part Number (none) -> RNCP0603FTD1K00
- R5: ALTIUM_VALUE 4.7k -> (none); DATASHEET LINK https://www.digikey.com/en/products/detail/panasonic-electr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 -> (none); MANUFACTURER Panasonic Electronic Components -> (none); MANUFACTURER PART NUMBER ERJ-3EKF4701V -> (none); OPERATING TEMPERATURE -55°C ~ 155°C -> (none); PACKAGE / CASE 0603 (1608 Metric) -> (none); Part Number (none) -> ERJ-3EKF4701V
- SW2: COMPONENTLINK1DESCRIPTION Upverter -> (none); COMPONENTLINK1URL https://upverter.com/upn/revision/12a774d2564c312a/ -> (none); COMPONENTLINK2DESCRIPTION Datasheet -> (none); COMPONENTLINK2URL http://www.omron.com/ecb/products/pdf/en-a6s.pdf -> (none); DIGIKEY DESCRIPTION SWITCH SLIDE DIP SPST 25MA 24V -> (none); DIGIKEY PART NUMBER A6S-1104-PH-ND -> (none); HELPURL https://upverter.com/upn/revision/12a774d2564c312a/ -> (none); LEAD FREE yes -> (none); MANUFACTURER Omron -> (none); MOUSER PART NUMBER 653-A6S1104PH -> (none); PACKAGE SMT_SW -> (none); PART NUMBER A6S-1104-PH -> (none); PRICE 1.25010001648 -> (none); Part Number (none) -> A6S-1104-PH; ROHS TRUE -> (none); SUPPLIER 1 Digi-Key -> (none); SUPPLIER 2 Mouser -> (none); SUPPLIER PART NUMBER 1 A6S-1104-PH-ND -> (none); SUPPLIER PART NUMBER 2 653-A6S1104PH -> (none); TEMPERATURE -20°C to +70°C -> (none); TEMPERATURE RANGE HIGH +70°C -> (none); TEMPERATURE RANGE LOW -20°C -> (none); VOLTAGE 24V -> (none)
- U1: DATASHEET LINK https://www.digikey.com/en/products/detail/texas-instrument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 -> (none); MANUFACTURER Texas Instruments -> (none); MANUFACTURER PART NUMBER OPA1604AIPWR -> (none); OPERATING TEMPERATURE -40°C ~ 85°C -> (none); PACKAGE / CASE 14-TSSOP -> (none); Part Number (none) -> OPA1604AIPWR

Commit message: Ready for review
Parts:
- removed SW2: Switch_Omron_A6S-1104-PH_eec, AltiumImports:Omron_A6S-1104-PH_0, symbol AcousticsSingleChannel-altium-import:BufferBiasAmp_1_Switch_Omron_A6S-1104-PH_e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
Connections:
- net BUF_IN: now also C2.2, U1.3 (IN_A+)
- net Mode_Sel: now reaches R21.2, R5.2
- net VCC renamed +3.3V

Commit message: Ready for Review.
Connections:
- net AGND: now also U1.5 (IN_B+); no longer U1.12 (IN_D+)
- net BBAmp_IN: now also U1.7 (OUT_B); no longer U1.14 (OUT_D)
- net at R2.1, R4.2: now also U1.6 (IN_B-); no longer U1.13 (IN_D-)
- net +3.3V renamed +5V
