File: OutputAmplifier.kicad_sch (KiCad schematic)
At the start: 7 parts, among them SW1 416131160803, U3 LTC6910-3CTS8#TRPBF

Commit message: Cleanup symbol table
Parts:
- C11: @ QTY 0 -> (none); ALTIUM_VALUE 1µF -> (none); APPLICATIONS Automotive -> (none); DATASHEETS http://www.murata.com/~/media/webrenewal/support/library/ca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 -> (none); DIGI-KEY PART NUMBER 490-5241-1-ND -> (none); FACTORY STOCK 0 -> (none); FEATURES - -> (none); HEIGHT - SEATED (MAX) - -> (none); IMAGE //media.digikey.com/Renders/Murata%20Renders/0603%28GCM188%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 -> (none); LEAD SPACING - -> (none); LEAD STYLE - -> (none); MANUFACTURER Murata Electronics North America -> (none); MINIMUM QUANTITY 1 -> (none); MOUNTING TYPE Surface Mount, MLCC -> (none); OPERATING TEMPERATURE -55°C ~ 125°C -> (none); PACKAGE / CASE 0603 (1608 Metric) -> (none); PACKAGING Cut Tape (CT) -> (none); PART NUMBER GCM188R71C105KA64D -> (none); PART STATUS Active -> (none); Part Number (none) -> GCM188R71C105KA64D; QUANTITY AVAILABLE 9243 -> (none); RATINGS AEC-Q200 -> (none); SERIES GCM -> (none); SIZE / DIMENSION 0.063" L x 0.031" W (1.60mm x 0.80mm) -> (none); TEMPERATURE COEFFICIENT X7R -> (none); THICKNESS (MAX) 0.035" (0.90mm) -> (none); TOLERANCE ±10% -> (none); UNIT PRICE (USD) 0.24 -> (none); VOLTAGE 16V -> (none)
- C12: @ QTY 0 -> (none); ALTIUM_VALUE 0.10µF -> (none); APPLICATIONS Automotive, Boardflex Sensitive -> (none); DATASHEETS http://www.murata.com/~/media/webrenewal/support/library/ca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 -> (none); DIGI-KEY PART NUMBER 490-5796-1-ND -> (none); FACTORY STOCK 0 -> (none); FEATURES Soft Termination -> (none); HEIGHT - SEATED (MAX) - -> (none); IMAGE //media.digikey.com/Renders/Murata%20Renders/0603%28LQG18%2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 -> (none); LEAD SPACING - -> (none); LEAD STYLE - -> (none); MANUFACTURER Murata Electronics North America -> (none); MINIMUM QUANTITY 1 -> (none); MOUNTING TYPE Surface Mount, MLCC -> (none); OPERATING TEMPERATURE -55°C ~ 125°C -> (none); PACKAGE / CASE 0603 (1608 Metric) -> (none); PACKAGING Cut Tape (CT) -> (none); PART NUMBER GCJ188R71C104KA01D -> (none); PART STATUS Active -> (none); Part Number (none) -> GCJ188R71C104KA01D; QUANTITY AVAILABLE 22473 -> (none); RATINGS AEC-Q200 -> (none); SERIES GCJ -> (none); SIZE / DIMENSION 0.063" L x 0.031" W (1.60mm x 0.80mm) -> (none); TEMPERATURE COEFFICIENT X7R -> (none); THICKNESS (MAX) 0.035" (0.90mm) -> (none); TOLERANCE ±10% -> (none); UNIT PRICE (USD) 0.21 -> (none); VOLTAGE 16V -> (none)
- R18, R19, R20: ALTIUM_VALUE 10k -> (none); DATASHEET LINK https://www.digikey.com/en/products/detail/stackpole-electr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 -> (none); MANUFACTURER Panasonic Electronic Components -> (none); MANUFACTURER PART NUMBER RNCP0603FTD10K0 -> (none); OPERATING TEMPERATURE -55°C ~ 155°C -> (none); PACKAGE / CASE 0603 (1608 Metric) -> (none); Part Number (none) -> RNCP0603FTD10K0
- SW1: DATASHEET LINK https://www.we-online.com/catalog/datasheet/416131160803.pdf -> (none); HEIGHT 2.65mm -> (none); MANUFACTURER_NAME Wurth Elektronik -> (none); MANUFACTURER_PART_NUMBER 416131160803 -> (none); MOUSER PART NUMBER 710-416131160803 -> (none); MOUSER PRICE/STOCK https://www.mouser.co.uk/ProductDetail/Wurth-Elektronik/416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 -> (none); Part Number (none) -> 416131160803
- U3: ALTIUM_VALUE N/A -> (none); DATASHEET LINK https://www.analog.com/media/en/technical-documentation/dat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 -> (none); MANUFACTURER Analog Devices Inc. -> (none); MANUFACTURER PART NUMBER LTC6910-3CTS8#TRMPBF -> (none); OPERATING TEMPERATURE 0°C ~ 70°C -> (none); PACKAGE / CASE TSOT-23-8 -> (none); Part Number (none) -> LTC6910-3CTS8#TRMPBF; ROHS Pb-Free -> (none)

Commit message: Update fixing local weirdness? Changed some trace widths
Parts:
- removed R18, R19, R20: 10k, AltiumImports:SMD-0603-RES, symbol AcousticsSingleChannel-altium-import:OutputAmplifier_0_ERJ-3EKF1002V
- removed SW1: 416131160803, AltiumImports:416131160803, symbol AcousticsSingleChannel-altium-import:OutputAmplifier_2_mirrored_416131160803
Connections:
- net G0 renamed G0_out
- net G1 renamed G1_out
- net G2 renamed G2_out

Commit message: Ready for review
Connections:
- net VCC renamed +3.3V

Commit message: Ready for Review.
Connections:
- net +3.3V renamed +5V
Changed lines of the file:
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@@
-	)
-	(symbol
-		(lib_id "power:+3.3V")
-		(at 81.28 119.38 0)
-		(unit 1)
-		(exclude_from_sim no)
-		(in_bom yes)
-		(on_board yes)
-		(dnp no)
-		(fields_autoplaced yes)
-		(property "Reference" "#PWR040"
-			(at 81.28 123.19 0)
-			(effects
-				(font
-					(size 1.27 1.27)
-				)
-				(hide yes)
-			)
-		)
-		(property "Value" "+3.3V"
-			(at 81.28 114.3 0)
-			(effects
-				(font
-					(size 1.27 1.27)
-				)
-			)
-		)
-		(property "Footprint" ""
-			(at 81.28 119.38 0)
-			(effects
-				(font
-					(size 1.27 1.27)
-				)
-				(hide yes)
-			)
-		)
-		(property "Datasheet" ""
-			(at 81.28 119.38 0)
-			(effects
-				(font
-					(size 1.27 1.27)
-				)
-				(hide yes)
-			)
-		)
-		(property "Description" "Power symbol creates a global label with name \"+3.3V\""
-			(at 81.28 119.38 0)
-			(effects
-				(font
-					(size 1.27 1.27)
-				)
-				(hide yes)
-			)
-		)
-		(pin "1"
-		)
-		(instances
-			(project "AcousticsSingleChannel"
-				(path "/8b2368f6-513e-479c-aa25-8a2dd439cbb4/3e62cd89-d47d-4712-b27b-57e94837f59d"
-					(reference "#PWR040")
-					(unit 1)
-				)
-			)
-		)
 	)
 	(symbol
@@
 					(unit 1)
 				)
+			)
+		)
+	)
+	(symbol
+		(lib_id "power:+5V")
+		(at 81.28 119.38 0)
+		(unit 1)
+		(exclude_from_sim no)
+		(in_bom yes)
+		(on_board yes)
+		(dnp no)
+		(property "Reference" "#PWR029"
+			(at 81.28 123.19 0)
+			(effects
+				(font
+					(size 1.27 1.27)
+				)
+				(hide yes)
+			)
+		)
+		(property "Value" "+5V"
+			(at 77.978 116.84 0)
+			(effects
+				(font
+					(size 1.27 1.27)
+				)
+			)
+		)
+		(property "Footprint" ""
+			(at 81.28 119.38 0)
+			(effects
+				(font
+					(size 1.27 1.27)
+				)
+				(hide yes)
+			)
+		)
+		(property "Datasheet" ""
+			(at 81.28 119.38 0)
+			(effects
+				(font
+					(size 1.27 1.27)
+				)
+				(hide yes)
+			)
+		)
+		(property "Description" "Power symbol creates a global label with name \"+5V\""
+			(at 81.28 119.38 0)
+			(effects
+				(font
+					(size 1.27 1.27)
+				)
+				(hide yes)
+			)
+		)
+		(pin "1"
+		)
+		(instances
+			(project "AcousticsSingleChannel"
+				(path "/8b2368f6-513e-479c-aa25-8a2dd439cbb4/3e62cd89-d47d-4712-b27b-57e94837f59d"
+					(reference "#PWR029")
+					(unit 1)
+				)
