File: AcousticsSingleChannel.kicad_sch (KiCad schematic)
At the start: 13 parts, among them J5 87233-3, J7 SAMTEC-SMH-103-02-X-S, J8 22-05-3021, U2 OPA1604AIPWR, U4 LTC1197LIMS8#PBF

Commit message: Fix various net and footprint issues
Connections:
- net Amp_Out renamed OutputAmplifier/Amp_Out
- net BBA IN renamed BufferBiasAmp/BBA_IN
Other:
- sheet Band Pass Filter ports: added BPF_IN, BPF_OUT; removed BPF IN, BPF OUT
- sheet BufferBiasAmp ports: added BBA_IN, BBA_OUT; removed BBA IN, BBA OUT
Changed lines of the file:
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@@
     (effects (font (size 1.27 1.27)) (justify left bottom))
   )
-  (label "BBA OUT" (at 68.58 111.76 0)
-    (effects (font (size 1.27 1.27)) (justify left bottom))
-  )
-  (label "Sig_Out" (at 200.66 96.52 270)
+  (label "Sig_Out" (at 200.66 96.52 270) (fields_autoplaced)
     (effects (font (size 1.27 1.27)) (justify right bottom))
-  )
-  (label "BPF OUT" (at 109.22 111.76 0)
-    (effects (font (size 1.27 1.27)) (justify left bottom))
-  )
-  (label "Amp_Out" (at 157.48 111.76 0)
-    (effects (font (size 1.27 1.27)) (justify left bottom))
-  )
-  (label "BBA IN" (at 25.4 111.76 0)
-    (effects (font (size 1.27 1.27)) (justify left bottom))
   )
   (symbol (lib_id "AcousticsSingleChannel-altium-import:GND") (at 182.88 134.62 180) (unit 1)
@@
       (effects (font (size 1.27 1.27)) (justify left bottom))
     )
-    (pin "BPF IN" input (at 78.74 111.76 180)
+    (pin "BPF_IN" input (at 78.74 111.76 180)
       (effects (font (size 1.27 1.27)) (justify left))
     )
-    (pin "BPF OUT" output (at 109.22 111.76 0)
+    (pin "BPF_OUT" output (at 109.22 111.76 0)
       (effects (font (size 1.27 1.27)) (justify right))
     )
@@
       (effects (font (size 1.27 1.27)) (justify left bottom))
     )
-    (pin "BBA IN" input (at 35.56 111.76 180)
+    (pin "BBA_IN" input (at 35.56 111.76 180)
       (effects (font (size 1.27 1.27)) (justify left))
     )
-    (pin "BBA OUT" output (at 68.58 111.76 0)
+    (pin "BBA_OUT" output (at 68.58 111.76 0)
       (effects (font (size 1.27 1.27)) (justify right))
     )

Commit message: Cleanup symbol table
Parts:
- C13: @ QTY 0 -> (none); ALTIUM_VALUE 1µF -> (none); APPLICATIONS General Purpose -> (none); DATASHEETS http://www.murata.com/~/media/webrenewal/support/library/ca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 -> (none); DIGI-KEY PART NUMBER 490-8271-1-ND -> (none); FACTORY STOCK 0 -> (none); FEATURES - -> (none); HEIGHT - SEATED (MAX) - -> (none); IMAGE //media.digikey.com/Renders/Murata%20Renders/ZRB-SERIES-040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 -> (none); LEAD SPACING - -> (none); LEAD STYLE - -> (none); MANUFACTURER Murata Electronics North America -> (none); MINIMUM QUANTITY 1 -> (none); MOUNTING TYPE Surface Mount, MLCC -> (none); OPERATING TEMPERATURE -55°C ~ 105°C -> (none); PACKAGE / CASE 0603 (1608 Metric) -> (none); PACKAGING Cut Tape (CT) -> (none); PART NUMBER GRM185C80J105KE26D -> (none); PART STATUS Active -> (none); Part Number (none) -> GRM185C80J105KE26D; QUANTITY AVAILABLE 11240 -> (none); RATINGS - -> (none); SERIES GRM -> (none); SIZE / DIMENSION 0.063" L x 0.031" W (1.60mm x 0.80mm) -> (none); TEMPERATURE COEFFICIENT X6S -> (none); THICKNESS (MAX) 0.020" (0.50mm) -> (none); TOLERANCE ±10% -> (none); UNIT PRICE (USD) 0.2 -> (none); VOLTAGE 6.3V -> (none)
- C14, C15: ALTIUM_VALUE 1µF -> (none); DATASHEET LINK https://www.digikey.com/en/products/detail/samsung-electro-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 -> (none); MANUFACTURER Samsung Electro-Mechanics -> (none); MANUFACTURER PART NUMBER CL10A105KA8NNNC -> (none); OPERATING TEMPERATURE -55°C ~ 125°C -> (none); PACKAGE / CASE 0603 (1608 Metric) -> (none); Part Number (none) -> CL10A105KA8NNNC
- C18: @ QTY 0 -> (none); ALTIUM_VALUE 2.2µF -> (none); APPLICATIONS Automotive -> (none); DATASHEETS http://www.murata.com/~/media/webrenewal/support/library/ca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 -> (none); DIGI-KEY PART NUMBER 490-5316-1-ND -> (none); FACTORY STOCK 0 -> (none); FEATURES - -> (none); HEIGHT - SEATED (MAX) - -> (none); IMAGE //media.digikey.com/Renders/Murata%20Renders/0603%28GCM188%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 -> (none); LEAD SPACING - -> (none); LEAD STYLE - -> (none); MANUFACTURER Murata Electronics North America -> (none); MINIMUM QUANTITY 1 -> (none); MOUNTING TYPE Surface Mount, MLCC -> (none); OPERATING TEMPERATURE -55°C ~ 125°C -> (none); PACKAGE / CASE 0603 (1608 Metric) -> (none); PACKAGING Cut Tape (CT) -> (none); PART NUMBER GCM188R70J225KE22D -> (none); PART STATUS Active -> (none); Part Number (none) -> GCM188R70J225KE22D; QUANTITY AVAILABLE 20695 -> (none); RATINGS AEC-Q200 -> (none); SERIES GCM -> (none); SIZE / DIMENSION 0.063" L x 0.031" W (1.60mm x 0.80mm) -> (none); TEMPERATURE COEFFICIENT X7R -> (none); THICKNESS (MAX) 0.035" (0.90mm) -> (none); TOLERANCE ±10% -> (none); UNIT PRICE (USD) 0.23 -> (none); VOLTAGE 6.3V -> (none)
- D1: ALTIUM_VALUE 1.9V -> (none); DATASHEET LINK https://www.mouser.com/ProductDetail/Wurth-Elektronik/15008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 -> (none); MANUFACTURER Wurth Elektronics -> (none); MANUFACTURER PART NUMBER 150080SS75000 -> (none); OPERATING TEMPERATURE -40to85degC -> (none); PACKAGE / CASE 0805 (2012 Metric) -> (none); Part Number (none) -> 150080SS75000; ROHS Pb-Free -> (none)
- J5: ALTIUM_VALUE * -> (none); AVAILABILITY Unavailable -> (none); MF {'manufacturer': u'TE Connectivity'} -> (none); MP 87233-3 -> (none); PACKAGE None -> (none); PRICE None -> (none); Part Number (none) -> 87233-3
- J7: ALTIUM_VALUE * -> (none); AVAILABILITY Unavailable -> (none); MF {'manufacturer': u'Samtec'} -> (none); MP SAMTEC-SMH-103-02-X-S -> (none); PACKAGE None -> (none); PRICE None -> (none); Part Number (none) -> SAMTEC-SMH-103-02-X-S
- J8: APPROVALS UL -> (none); COLOR White -> (none); CONTACT MATERIAL Brass -> (none); CONTACT MATING LENGTH 0.264inch -> (none); CONTACT PLATING Tin -> (none); CONTACT RESISTANCE 10mR -> (none); CONTACT TYPE Male Pin -> (none); CURRENT RATING 4A -> (none); DEPTH 12.83mm -> (none); FASTENING TYPE Friction -> (none); FLAMMABILITY RATING UL94 V-0 -> (none); GENDER Male -> (none); GLOW WIRE COMPLIANT Non-compliant -> (none); HALOGEN FREE Low Halogen -> (none); HEIGHT 6.35mm -> (none); HOUSING COLOR White -> (none); HOUSING MATERIAL Nylon -> (none); LEAD FREE Lead Free -> (none); LENGTH 5.08mm -> (none); MAX CURRENT RATING 4A -> (none); MAX OPERATING TEMPERATURE 75°C -> (none); MAX VOLTAGE RATING (AC) 250V -> (none); MIN OPERATING TEMPERATURE 0°C -> (none); MOUNT Through Hole -> (none); NUMBER OF CIRCUITS 2 -> (none); NUMBER OF CONTACTS 2 -> (none); NUMBER OF POSITIONS 2 -> (none); NUMBER OF ROWS 1 -> (none); ORIENTATION Right Angle -> (none); PACKAGE QUANTITY 3000 -> (none); PACKAGING Bulk -> (none); PITCH 2.54mm -> (none); Part Number (none) -> 22-05-3021; RADIATION HARDENING No -> (none); SERIES KK® 7478 -> (none); TERMINATION Solder -> (none); VOLTAGE RATING 250V -> (none)
- R25: ALTIUM_VALUE 300 -> (none); DATASHEET LINK https://www.digikey.com/en/products/detail/panasonic-electr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 -> (none); MANUFACTURER Panasonic Electronic Components -> (none); MANUFACTURER PART NUMBER ERJ-3EKF3000V -> (none); OPERATING TEMPERATURE -55°C ~ 155°C -> (none); PACKAGE / CASE 0603 (1608 Metric) -> (none); Part Number (none) -> ERJ-3EKF3000V
- R26: @ QTY 1500 -> (none); ALTIUM_VALUE 750 -> (none); COMPOSITION Thick Film -> (none); DATASHEETS http://industrial.panasonic.com/www-cgi/jvcr13pz.cgi?E+PZ+3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 -> (none); DIGI-KEY PART NUMBER P750HCT-ND -> (none); FACTORY STOCK 0 -> (none); FAILURE RATE - -> (none); FEATURES Automotive AEC-Q200 -> (none); HEIGHT - SEATED (MAX) 0.022" (0.55mm) -> (none); IMAGE //media.digikey.com/Photos/Panasonic%20Photos/MFG_ERJ-P6W%2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 -> (none); MANUFACTURER Panasonic Electronic Components -> (none); MINIMUM QUANTITY 1 -> (none); NUMBER OF TERMINATIONS 2 -> (none); OPERATING TEMPERATURE -55°C ~ 155°C -> (none); PACKAGE / CASE 0603 (1608 Metric) -> (none); PACKAGING Cut Tape (CT) -> (none); PART NUMBER ERJ-3EKF7500V -> (none); PART STATUS Active -> (none); POWER (WATTS) 0.1W, 1/10W -> (none); Part Number (none) -> ERJ-3EKF7500V; QUANTITY AVAILABLE 102837 -> (none); SERIES ERJ -> (none); SIZE / DIMENSION 0.063" L x 0.031" W (1.60mm x 0.80mm) -> (none); SUPPLIER DEVICE PACKAGE 0603 -> (none); TEMPERATURE COEFFICIENT ±100ppm/°C -> (none); TOLERANCE ±1% -> (none); UNIT PRICE (USD) 0.00379 -> (none)
- R27: @ QTY 1500 -> (none); ALTIUM_VALUE 1k -> (none); COMPOSITION Thick Film -> (none); DATASHEETS http://industrial.panasonic.com/www-cgi/jvcr13pz.cgi?E+PZ+3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 -> (none); DIGI-KEY PART NUMBER P1.00KHCT-ND -> (none); FACTORY STOCK 0 -> (none); FAILURE RATE - -> (none); FEATURES Automotive AEC-Q200 -> (none); HEIGHT - SEATED (MAX) 0.022" (0.55mm) -> (none); IMAGE //media.digikey.com/Photos/Panasonic%20Photos/MFG_ERJ-P6W%2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 -> (none); MANUFACTURER Panasonic Electronic Components -> (none); MINIMUM QUANTITY 1 -> (none); NUMBER OF TERMINATIONS 2 -> (none); OPERATING TEMPERATURE -55°C ~ 155°C -> (none); PACKAGE / CASE 0603 (1608 Metric) -> (none); PACKAGING Cut Tape (CT) -> (none); PART NUMBER ERJ-3EKF1001V -> (none); PART STATUS Active -> (none); POWER (WATTS) 0.1W, 1/10W -> (none); Part Number (none) -> ERJ-3EKF1001V; QUANTITY AVAILABLE 5218845 -> (none); SERIES ERJ -> (none); SIZE / DIMENSION 0.063" L x 0.031" W (1.60mm x 0.80mm) -> (none); SUPPLIER DEVICE PACKAGE 0603 -> (none); TEMPERATURE COEFFICIENT ±100ppm/°C -> (none); TOLERANCE ±1% -> (none); UNIT PRICE (USD) 0.00379 -> (none)
- U2: DATASHEET LINK https://www.digikey.com/en/products/detail/texas-instrument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 -> (none); MANUFACTURER Texas Instruments -> (none); MANUFACTURER PART NUMBER OPA1604AIPWR -> (none); OPERATING TEMPERATURE -40°C ~ 85°C -> (none); PACKAGE / CASE 14-TSSOP -> (none); Part Number (none) -> OPA1604AIPWR
- U4: CASE/PACKAGE MSOP -> (none); INTEGRAL NONLINEARITY (INL) 1LSB -> (none); INTERFACE SPI -> (none); LEAD FREE Lead Free -> (none); MAX OPERATING TEMPERATURE 85°C -> (none); MAX POWER DISSIPATION 25mW -> (none); MAX SUPPLY VOLTAGE 4V -> (none); MIN OPERATING TEMPERATURE -40°C -> (none); MIN SUPPLY VOLTAGE 2.7V -> (none); MOUNT Surface Mount -> (none); NUMBER OF BITS 10 -> (none); NUMBER OF CONVERTERS 1 -> (none); NUMBER OF ELEMENTS 1 -> (none); NUMBER OF PINS 8 -> (none); OPERATING SUPPLY VOLTAGE 3V -> (none); PACKAGE QUANTITY 50 -> (none); PACKAGING Rail/Tube -> (none); POLARITY Unipolar -> (none); POWER DISSIPATION 500mW -> (none); Part Number (none) -> LTC1197LIMS8#PBF; RESOLUTION 10b -> (none); ROHS COMPLIANT Yes -> (none); SAMPLING RATE 250000S/s -> (none); SUPPLY TYPE Single -> (none)

Commit message: Update fixing local weirdness? Changed some trace widths
Parts:
- removed J7: SAMTEC-SMH-103-02-X-S, AltiumImports:SAMTEC-SMH-103-02-X-S, symbol AcousticsSingleChannel-altium-import:root_2_SAMTEC-SMH-103-02-X-S
- added J1, J2: 87233-3, AltiumImports:TE_87233-3, symbol AcousticsSingleChannel-altium-import:root_2_87233-3
- renumbered J5 to J3
Connections:
- net at R26.1, R27.2: now also J2.1
- net at U4.7 (CLK): now also J2.2
- net at U4.1 (~{CS}): now also J2.3
- new net OutputAmplifier/G0_out: J1.1
- new net OutputAmplifier/G1_out: J1.2
- new net OutputAmplifier/G2_out: J1.3
Other:
- sheet OutputAmplifier ports: added G0_out, G1_out, G2_out; removed none
- note added: "C14 - VCC goes to J3 C15 - GND goes to J3"
- note added: "LED Power Indicator"
Changed lines of the file:
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@@
     (stroke (width 0.254) (type default))
+  )
+  (wire (pts (xy 138.43 82.55) (xy 34.29 82.55))
+    (stroke (width 0) (type default))
   )
   (wire (pts (xy 22.86 106.68) (xy 20.32 106.68))
@@
     (stroke (width 0.254) (type default))
   )
+  (wire (pts (xy 138.43 101.6) (xy 138.43 82.55))
+    (stroke (width 0) (type default))
+  )
+  (wire (pts (xy 132.08 167.64) (xy 210.82 167.64))
+    (stroke (width 0) (type default))
+  )
   (wire (pts (xy 182.88 142.24) (xy 182.88 134.62))
     (stroke (width 0.254) (type default))
@@
     (stroke (width 0.254) (type default))
   )
-  (wire (pts (xy 172.72 149.86) (xy 182.88 149.86))
+  (wire (pts (xy 171.45 149.86) (xy 182.88 149.86))
     (stroke (width 0.254) (type default))
   )
@@
     (stroke (width 0.254) (type default))
   )
-  (wire (pts (xy 210.82 167.64) (xy 210.82 139.7))
-    (stroke (width 0.254) (type default))
-  )
-  (wire (pts (xy 152.4 167.64) (xy 210.82 167.64))
-    (stroke (width 0.254) (type default))
+  (wire (pts (xy 140.97 80.01) (xy 34.29 80.01))
+    (stroke (width 0) (type default))
   )
   (wire (pts (xy 198.12 104.14) (xy 198.12 99.06))
@@
     (stroke (width 0.254) (type default))
   )
-  (wire (pts (xy 172.72 165.1) (xy 172.72 149.86))
-    (stroke (width 0.254) (type default))
+  (wire (pts (xy 135.89 85.09) (xy 135.89 101.6))
+    (stroke (width 0) (type default))
   )
   (wire (pts (xy 27.94 142.24) (xy 27.94 147.32))
@@
     (stroke (width 0.254) (type default))
   )
+  (wire (pts (xy 34.29 85.09) (xy 135.89 85.09))
+    (stroke (width 0) (type default))
+  )
   (wire (pts (xy 198.12 139.7) (xy 198.12 142.24))
     (stroke (width 0.254) (type default))
@@
     (stroke (width 0.254) (type default))
   )
+  (wire (pts (xy 132.08 170.18) (xy 171.45 170.18))
+    (stroke (width 0) (type default))
+  )
   (wire (pts (xy 33.02 152.4) (xy 33.02 144.78))
     (stroke (width 0.254) (type default))
   )
-  (wire (pts (xy 152.4 165.1) (xy 172.72 165.1))
-    (stroke (width 0.254) (type default))
-  )
   (wire (pts (xy 175.26 86.36) (xy 175.26 83.82))
     (stroke (width 0.254) (type default))
   )
+  (wire (pts (xy 171.45 149.86) (xy 171.45 170.18))
+    (stroke (width 0) (type default))
+  )
   (wire (pts (xy 185.42 93.98) (xy 187.96 93.98))
     (stroke (width 0.254) (type default))
   )
+  (wire (pts (xy 140.97 101.6) (xy 140.97 80.01))
+    (stroke (width 0) (type default))
+  )
   (wire (pts (xy 210.82 99.06) (xy 210.82 104.14))
     (stroke (width 0.254) (type default))
@@
     (stroke (width 0.254) (type default))
   )
+  (wire (pts (xy 210.82 139.7) (xy 210.82 167.64))
+    (stroke (width 0) (type default))
+  )
   (wire (pts (xy 187.96 93.98) (xy 200.66 93.98))
     (stroke (width 0.254) (type default))
   )
-  (wire (pts (xy 167.64 162.56) (xy 167.64 144.78))
+  (wire (pts (xy 167.64 165.1) (xy 167.64 144.78))
     (stroke (width 0.254) (type default))
   )
@@
     (stroke (width 0.254) (type default))
   )
-  (wire (pts (xy 152.4 162.56) (xy 167.64 162.56))
+  (wire (pts (xy 132.08 165.1) (xy 167.64 165.1))
     (stroke (width 0.254) (type default))
   )
@@
   )
   (text "Close to pin 3" (at 127 139.7 0)
+    (effects (font (size 1.27 1.27)) (justify left bottom))
+  )
+  (text "C14 - VCC goes to J3\nC15 - GND goes to J3" (at 17.78 177.8 0)
+    (effects (font (size 1.27 1.27)) (justify left bottom))
+  )
+  (text "LED Power Indicator" (at 59.69 175.26 0)
     (effects (font (size 1.27 1.27)) (justify left bottom))
   )
@@
   (symbol (lib_id "AcousticsSingleChannel-altium-import:root_2_87233-3") (at 12.7 147.32 0) (unit 1)
     (in_bom yes) (on_board yes) (dnp no)
-    (property "Reference" "J5" (at 7.62 142.24 0)
+    (property "Reference" "J3" (at 7.62 142.24 0)
       (effects (font (size 1.27 1.27)) (justify left bottom))
     )
@@
       (project "AcousticsSingleChannel"
         (path "/8b2368f6-513e-479c-aa25-8a2dd439cbb4"
-          (reference "J5") (unit 1)
+          (reference "J3") (unit 1)
         )
       )
@@
         (path "/8b2368f6-513e-479c-aa25-8a2dd439cbb4"
           (reference "#PWR0101") (unit 1)
-        )
-      )
-    )
-  )
-  (symbol (lib_id "AcousticsSingleChannel-altium-import:root_2_SAMTEC-SMH-103-02-X-S") (at 147.32 167.64 0) (unit 1)
-    (in_bom yes) (on_board yes) (dnp no)
-    (property "Reference" "J7" (at 121.92 149.86 0)
-      (effects (font (size 1.27 1.27)) (justify left bottom))
-    )
-    (property "Value" "SAMTEC-SMH-103-02-X-S" (at 121.92 175.26 0)
-      (effects (font (size 1.27 1.27)) (justify left bottom))
-    )
-    (property "Footprint" "AltiumImports:SAMTEC-SMH-103-02-X-S" (at 147.32 167.64 0)
-      (effects (font (size 1.27 1.27)) hide)
-    )
-    (property "Datasheet" "" (at 147.32 167.64 0)
-      (effects (font (size 1.27 1.27)) hide)
-    )
-    (property "Part Number" "SAMTEC-SMH-103-02-X-S" (at 147.32 167.64 0)
-      (effects (font (size 1.27 1.27)) hide)
-    )
-    (pin "1")
-    (pin "2")
-    (pin "3")
-    (instances
-      (project "AcousticsSingleChannel"
-        (path "/8b2368f6-513e-479c-aa25-8a2dd439cbb4"
-          (reference "J7") (unit 1)
         )
       )
@@
     )
   )
+  (symbol (lib_id "AcousticsSingleChannel-altium-import:root_2_87233-3") (at 121.92 167.64 0) (unit 1)
+    (in_bom yes) (on_board yes) (dnp no)
+    (property "Reference" "J2" (at 116.84 162.56 0)
+      (effects (font (size 1.27 1.27)) (justify left bottom))
+    )
+    (property "Value" "87233-3" (at 116.84 175.26 0)
+      (effects (font (size 1.27 1.27)) (justify left bottom))
+    )
+    (property "Footprint" "AltiumImports:TE_87233-3" (at 121.92 167.64 0)
+      (effects (font (size 1.27 1.27)) hide)
+    )
+    (property "Datasheet" "" (at 121.92 167.64 0)
+      (effects (font (size 1.27 1.27)) hide)
+    )
+    (property "Part Number" "87233-3" (at 121.92 167.64 0)
+      (effects (font (size 1.27 1.27)) hide)
+    )
+    (pin "1")
+    (pin "2")
+    (pin "3")
+    (instances
+      (project "AcousticsSingleChannel"
+        (path "/8b2368f6-513e-479c-aa25-8a2dd439cbb4"
+          (reference "J2") (unit 1)
+        )
+      )
+    )
+  )
   (symbol (lib_id "AcousticsSingleChannel-altium-import:VCC") (at 55.88 149.86 180) (unit 1)
     (in_bom yes) (on_board yes) (dnp no)
@@
     )
   )
+  (symbol (lib_id "AcousticsSingleChannel-altium-import:root_2_87233-3") (at 24.13 82.55 0) (unit 1)
+    (in_bom yes) (on_board yes) (dnp no)
+    (property "Reference" "J1" (at 19.05 77.47 0)
+      (effects (font (size 1.27 1.27)) (justify left bottom))
+    )
+    (property "Value" "87233-3" (at 19.05 90.17 0)
+      (effects (font (size 1.27 1.27)) (justify left bottom))
+    )
+    (property "Footprint" "AltiumImports:TE_87233-3" (at 24.13 82.55 0)
+      (effects (font (size 1.27 1.27)) hide)
+    )
+    (property "Datasheet" "" (at 24.13 82.55 0)
+      (effects (font (size 1.27 1.27)) hide)
+    )
+    (property "Part Number" "87233-3" (at 24.13 82.55 0)
+      (effects (font (size 1.27 1.27)) hide)
+    )
+    (pin "1")
+    (pin "2")
+    (pin "3")
+    (instances
+      (project "AcousticsSingleChannel"
+        (path "/8b2368f6-513e-479c-aa25-8a2dd439cbb4"
+          (reference "J1") (unit 1)
+        )
+      )
+    )
+  )
   (symbol (lib_id "AcousticsSingleChannel-altium-import:GND") (at 152.4 137.16 0) (unit 1)
     (in_bom yes) (on_board yes) (dnp no)
@@
           (reference "#PWR0108") (unit 1)
         )
+      )
+    )
+  )
+  (sheet (at 119.38 101.6) (size 30.48 13.97) (fields_autoplaced)
+    (stroke (width 0.1524) (type solid) (color 128 0 0 1))
+    (fill (color 128 255 128 1.0000))
+    (property "Sheetname" "OutputAmplifier" (at 119.38 100.8884 0)
+      (effects (font (size 1.27 1.27)) (justify left bottom))
+    )
+    (property "Sheetfile" "OutputAmplifier.kicad_sch" (at 119.38 116.1546 0)
+      (effects (font (size 1.27 1.27)) (justify left top))
+    )
+    (pin "Amp_Out" output (at 149.86 111.76 0)
+      (effects (font (size 1.27 1.27)) (justify right))
+    )
+    (pin "G1_out" output (at 138.43 101.6 90)
+      (effects (font (size 1.27 1.27)) (justify right))
+    )
+    (pin "G0_out" output (at 135.89 101.6 90)
+      (effects (font (size 1.27 1.27)) (justify right))
+    )
+    (pin "G2_out" output (at 140.97 101.6 90)
+      (effects (font (size 1.27 1.27)) (justify right))
+    )
+    (pin "Amp_In" input (at 119.38 111.76 180)
+      (effects (font (size 1.27 1.27)) (justify left))
+    )
+    (instances
+      (project "AcousticsSingleChannel"
+        (path "/8b2368f6-513e-479c-aa25-8a2dd439cbb4" (page "5"))
       )
     )
@@
       )
     )
-  )
-  (sheet (at 119.38 106.68) (size 30.48 10.16) (fields_autoplaced)
-    (stroke (width 0) (type solid) (color 128 0 0 1))
-    (fill (color 128 255 128 1.0000))
-    (property "Sheetname" "OutputAmplifier" (at 119.38 104.14 0)
-      (effects (font (size 1.27 1.27)) (justify left bottom))
-    )
-    (property "Sheetfile" "OutputAmplifier.kicad_sch" (at 119.38 106.68 0)
-      (effects (font (size 1.27 1.27)) (justify left bottom))
-    )
-    (pin "Amp_In" input (at 119.38 111.76 180)
-      (effects (font (size 1.27 1.27)) (justify left))
-    )
-    (pin "Amp_Out" output (at 149.86 111.76 0)
-      (effects (font (size 1.27 1.27)) (justify right))
-    )
-    (instances
-      (project "AcousticsSingleChannel"
-        (path "/8b2368f6-513e-479c-aa25-8a2dd439cbb4" (page "4"))
-      )
-    )

Commit message: Ready for review
Parts:
- removed J1, J2, J3: 87233-3, AltiumImports:TE_87233-3, symbol AcousticsSingleChannel-altium-import:root_2_87233-3
- removed J8: 22-05-3021, AltiumImports:FP-22-05-3021-MFG, symbol AcousticsSingleChannel-altium-import:root_0_3bc925449376181038e59eaffc5286c
- removed U4: LTC1197LIMS8#PBF, AltiumImports:FP-MS8-8-05-08-1660-IPC_A, symbol AcousticsSingleChannel-altium-import:root_3_b4ff916109b4f52b6d17af6699a3653
- added C19: 1.5nF, AltiumImports:SMD-0603C, symbol AcousticsSingleChannel-altium-import:root_0_GRM185C80J105KE26D
- added J1: SSW-104-01-G-D, Accoustics:SAMTEC_SSW-104-01-G-D, symbol Accoustics:SSW-104-01-G-D
- added J2: TSW-104-07-F-D, Accoustics:SAMTEC_TSW-104-07-F-D, symbol Accoustics:TSW-104-07-F-D
- added R18: 25, AltiumImports:SMD-0603-RES, symbol AcousticsSingleChannel-altium-import:root_0_ERJ-3EKF7500V
- added TP1, TP2, TP3: 5005, Accoustics:KEYSTONE_5005, symbol Accoustics:5005
- added TP4: 5006, Accoustics:KEYSTONE_5006, symbol Accoustics:5006
- added U4: ADS7042IDCUR, Accoustics:DCU0008A_L, symbol Accoustics:ADS7042IDCUR
- C18: value 2.2µF -> 1µF
- R26: value 750 -> 0
- R27: value 1k -> 0; now not fitted
Connections:
- net AGND: now also J1.02
- net Band Pass Filter/BPF_IN: now also TP1.TP
- net Band Pass Filter/BPF_OUT: now also TP2.TP
- net GND: now also C19.2, J1.08, TP4.TP, U4.5 (AINM), U4.8 (GND)
- net Sig_Out: now also R18.1, TP3.TP
- net at R26.1, R27.2: now also J2.05
- net at R26.2: now also U4.3 (SDO)
- net VCC renamed +3.3V
- net +3.3V: now also J1.04, U4.1 (DVDD), U4.7 (AVDD)
- new net: C19.1, R18.2, U4.6 (AINP)
- new net: J2.07, U4.2 (SCLK)
- new net: J2.03, U4.4 (CS_N)
- new net +5V: J1.06
- new net G0_out: J1.01
- new net G1_out: J1.03
- new net G2_out: J1.05
- new net Hydro+: J1.07
- new net Mode_Sel: J2.08
- no-connect marks 0 -> 4
Other:
- sheet BufferBiasAmp ports: added Mode_Sel; removed none
- note added: "C14 - VCC goes to J1 C15 - GND goes to J1"
- note added: "Close to pin 1"
- note added: "Clsoe to pin 7"
- note removed: "C14 - VCC goes to J3 C15 - GND goes to J3"
- note removed: "Close to pin 3"
- note removed: "Clsoe to pin 4"
- moved on the sheet: C13, C14, C15, C18, D1, R25

Commit message: Ready for Review.
Parts:
- removed C19: 1.5nF, AltiumImports:SMD-0603C, symbol AcousticsSingleChannel-altium-import:root_0_GRM185C80J105KE26D
- removed R18: 25, AltiumImports:SMD-0603-RES, symbol AcousticsSingleChannel-altium-import:root_0_ERJ-3EKF7500V
- removed TP2: 5005, Accoustics:KEYSTONE_5005, symbol Accoustics:5005
- removed U4: ADS7042IDCUR, Accoustics:DCU0008A_L, symbol Accoustics:ADS7042IDCUR
- added C3, C4: 1µF, AltiumImports:SMD-0603C, symbol AcousticsSingleChannel-altium-import:root_0_GCM188R70J225KE22D
- added C5: 0F, AltiumImports:SMD-0603C, symbol AcousticsSingleChannel-altium-import:root_0_GRM185C80J105KE26D
- added C6: 1µF, AltiumImports:SMD-0603C, symbol AcousticsSingleChannel-altium-import:root_2_GCM188R71C105KA64D
- added C7: .1µF, AltiumImports:SMD-0603C, symbol AcousticsSingleChannel-altium-import:root_2_GCM188R71C105KA64D
- added R6: 0, AltiumImports:SMD-0603-RES, symbol AcousticsSingleChannel-altium-import:root_0_ERJ-3EKF7500V
- added U2: ADS127L21IRUKT, Accoustics:WQFN20_RUK_TEX, symbol Accoustics:ADS127L21IRUKT
- C13: value 1µF -> .1µF
- renumbered U2 to U1
Connections:
- net +3.3V: now also C6.2, C7.2, U2.13 (IOVDD); no longer C13.1, C14.2, C15.2, C18.1, R25.2, U1.4 (V+)
- net +5V: now also C13.1, C14.2, C15.2, C18.1, R25.2, U1.4 (V+), U2.19 (AVDD2), U2.20 (AVDD1), U2.4 (REFP)
- net GND: now also C3.2, C4.2, C5.1, C6.1, C7.1, U2.14 (DGND), U2.17 (AVSS), U2.2 (AINN), U2.5 (REFN)
- net OutputAmplifier/Amp_Out: now also U1.12 (IN_D+); no longer U1.5 (IN_B+)
- net Sig_Out: now also U1.13 (IN_D-), U1.14 (OUT_D), R6.1; no longer U1.6 (IN_B-), U1.7 (OUT_B)
- net at R26.1, R27.2: now also J2.06; no longer J2.05
- net DOUT: now reaches R26.2
- net DOUT: now also U2.10 (SDO/*DRDY)
- net START: now reaches J2.07
- net START: now also U2.16 (START)
- net SCLK: now reaches J2.03
- net SCLK: now also U2.9 (SCLK)
- net CS: now reaches J2.01
- net CS: now also U2.7 (*CS)
- net RESET: now reaches J2.02
- net RESET: now also U2.6 (*RESET)
- net SDI: now reaches J2.04
- net SDI: now also U2.8 (SDI)
- net Band Pass Filter/BPF_IN renamed BufferBiasAmp/BBA_OUT
- new net: C5.2, R6.2, U2.1 (AINP)
- new net: C4.1, U2.15 (CAPD)
- new net: C3.1, U2.18 (CAPA)
- new net CLK: J2.05, U2.12 (CLK)
- no-connect marks 4 -> 3
Other:
- removed sheet Band Pass Filter
- note added: "C6 and C7 close to pin 13"
- note added: "Close to pin 19"
- note added: "Clsoe to pin 20"
- note removed: "Close to pin 1"
- note removed: "Clsoe to pin 7"
- moved on the sheet: C13, C18, R26, R27

Commit message: Ready for Review.
Parts:
- added R7, R8: 0, AltiumImports:SMD-0603-RES, symbol AcousticsSingleChannel-altium-import:root_0_ERJ-3EKF7500V
- added U4: mcp1416t-e/ot, Accoustics:SOT-23-5_MC_MCH-M, symbol Accoustics:mcp1416t-e_ot
Connections:
- net +3.3V: now also R7.1
- net +5V: now also R8.1
- net GND: now also U4.4 (GND)
- net Mode_Sel: now also U4.3 (IN)
- new net: R7.2, R8.2, U4.2 (VDD)
- new net Mode_Sel_Out: U4.5 (OUT)
